File: hardware/kicad/Gesture Glove/Gesture Glove.kicad_sch (KiCad schematic)
At the start: 41 parts, among them U1 XIAO-nRF52840-SMD, U2 Adafruit-BNO085, U3 A13xxxLHxx-x, U4 A13xxxLHxx-x, U5 A13xxxLHxx-x, U6 MCP6004, U7 MCP6002-xSN, U8 LMR14020SQDDARQ1, U9 TPS7A20xxxDBV

Commit message: Fix to Libraries
Connections:
- net 3VO_HES2 is gone; now on net 3V3_HES2: U6.6 (-), U6.7
- net 3V0_HES1 renamed 3V3_HES1
- net 3V0_HES2 renamed 3V3_HES2
- net 3V0_HES3 renamed 3V3_HES3
Changed lines of the file:
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@@
 		(title "Gesture Glove Full Schematic")
 		(date "2026-10-22")
-		(rev "1.09")
+		(rev "1.10")
 		(company "N-TAIL")
 	)
@@
 		)
 	)
-	(label "3V0_HES2"
+	(label "3V3_HES2"
 		(at 56.515 163.195 90)
 		(effects
@@
 		)
 	)
-	(label "3VO_HES2"
+	(label "3V3_HES2"
 		(at 61.595 133.985 180)
 		(effects
@@
 		)
 	)
-	(label "3V0_HES1"
+	(label "3V3_HES1"
 		(at 36.195 133.985 180)
 		(effects
@@
 		)
 	)
-	(label "3V0_HES1"
+	(label "3V3_HES1"
 		(at 15.875 163.195 90)
 		(effects
@@
 		)
 	)
-	(label "3V0_HES3"
+	(label "3V3_HES3"
 		(at 86.995 133.985 180)
 		(effects
@@
 		)
 	)
-	(label "3V0_HES3"
+	(label "3V3_HES3"
 		(at 97.155 163.195 90)
 		(effects
